Commit message: Rocket moves and is orange

File: dev_ws/src/trackingplatform/description/rocket.urdf.xacro (robot description, xacro)
@@ -2,22 +2,35 @@
 <robot name="rocket">
     <link name="base_link">
+    </link>
+    <joint name="rocket_joint" type="fixed">
+        <origin xyz="0 0 0" rpy="0 0 0"/>
+        <parent link="base_link"/>
+        <child link="rocket"/>
+    </joint>
+    <link name="rocket">
         <inertial>
-            <origin xyz="0 0 0" rpy="0 0 0"/>
-            <mass value="0.01" />
-            <inertia ixx="7.58333333333e-06" ixy="0.0" ixz="0.0" iyy="7.58333333333e-06" iyz="0.0" izz="1.25e-05"/>
-        </inertial>
-        <collision>
-            <origin rpy="0 0 0" xyz="0 0 0"/>
-            <geometry>
-                <box size="0.5 0.5 0.5"/>
-            </geometry>
-        </collision>
-        <visual>
-            <origin rpy="1.5708 0 0" xyz="0 0 0"/>
-            <geometry>
-                <mesh filename="/home/marcus/rockettrackingplatform/dev_ws/src/trackingplatform/models/Example.stl" scale="0.001 0.001 0.001"/>
-                <!-- <box size="1 1 1"/> -->
-            </geometry>
-        </visual>
+                    <origin xyz="0 0 0" rpy="0 0 0"/>
+                    <mass value="0.01" />
+                    <inertia ixx="7.58333333333e-06" ixy="0.0" ixz="0.0" iyy="7.58333333333e-06" iyz="0.0" izz="1.25e-05"/>
+                </inertial>
+                <collision>
+                    <origin rpy="0 0 0" xyz="0 0 0"/>
+                    <geometry>
+                        <box size="0.2 0.2 0.2"/>
+                    </geometry>
+                </collision>
+                <visual>
+                    <origin rpy="1.5708 0 0" xyz="0 0 0"/>
+                    <geometry>
+                        <mesh filename="/home/marcus/rockettrackingplatform/dev_ws/src/trackingplatform/models/Example.stl" scale="0.001 0.001 0.001"/>
+                        <!-- <box size="1 1 1"/> -->
+                        <material name="orange">
+                            <color rgba="1 0.3 0.1 1"/>
+                        </material>
+                    </geometry>
+                </visual>
     </link>
+    <gazebo reference="rocket">
+        <material>Gazebo/Orange</material>
+    </gazebo>
 </robot>

Commit message: Updated rocket location STL find
should find the model no-matter where

File: dev_ws/src/trackingplatform/description/rocket.urdf.xacro (robot description, xacro)
@@ -11,11 +11,11 @@
         <inertial>
                     <origin xyz="0 0 0" rpy="0 0 0"/>
-                    <mass value="0.01" />
-                    <inertia ixx="7.58333333333e-06" ixy="0.0" ixz="0.0" iyy="7.58333333333e-06" iyz="0.0" izz="1.25e-05"/>
+                    <mass value="0.120" />
+                    <inertia ixx="7.58333333333e-06" ixy="0.0" ixz="0.0" iyy="7.58333333333e-06" iyz="0.0" izz="1.25e-05"/> <!-- This is actually wrong for this rocket -->
                 </inertial>
                 <collision>
                     <origin rpy="0 0 0" xyz="0 0 0"/>
                     <geometry>
-                        <box size="0.2 0.2 0.2"/>
+                        <box size="0.1 0.1 0.1"/>
                     </geometry>
                 </collision>
@@ -23,5 +23,5 @@
                     <origin rpy="1.5708 0 0" xyz="0 0 0"/>
                     <geometry>
-                        <mesh filename="/home/marcus/rockettrackingplatform/dev_ws/src/trackingplatform/models/Example.stl" scale="0.001 0.001 0.001"/>
+                        <mesh filename="$(find trackingplatform)/models/Example.stl" scale="0.001 0.001 0.001"/>
                         <!-- <box size="1 1 1"/> -->
                         <material name="orange">
@@ -34,3 +34,22 @@
         <material>Gazebo/Orange</material>
     </gazebo>
+    <gazebo>
+        <plugin name="gazebo_ros_joint_state_publisher"
+            filename="libgazebo_ros_joint_state_publisher.so">
+            <update_rate>20</update_rate>
+            <joint_name>rocket_joint</joint_name>
+        </plugin>
+    </gazebo>
+    <!-- This plugin will read a JointTrajectory message from the /set_joint_trajectory topic
+            and move the machine accordingly. It's a bit clunky but it works. -->
+    <!-- You'll probably want to add damping to the joints to stop them it flopping around.
+            e.g. <dynamics damping="10.0" friction="10.0"/> -->
+    <!-- Here's an example message to publish to test it:
+            ros2 topic pub -1 /set_joint_trajectory trajectory_msgs/msg/JointTrajectory  '{header: {frame_id: world}, joint_names: [slider_joint, arm_joint], points: [  {positions: {0.8,0.6}} ]}' -->
+    <gazebo>
+        <plugin name="gazebo_ros_joint_pose_trajectory"
+            filename="libgazebo_ros_joint_pose_trajectory.so">
+            <update_rate>2</update_rate>
+        </plugin>
+    </gazebo>
 </robot>
