Commit message: Added launch script for controller

File: dev_ws/src/trackingplatform/description/robot.urdf.xacro (robot description, xacro)
@@ -6,9 +6,10 @@
     <!-- This will include all the contents of example_include.xacro first. Go check it out! -->
     <xacro:include filename="include.xacro" />
+    <xacro:include filename="ros2_control.xacro" />
     <!-- This first link called "world" is empty -->
     <link name="world"></link>
     <!-- A simple fixed joint from our empty world link, to our base. -->
     <!-- The base origin is offset from the world origin. -->
-        <joint name="base_joint" type="fixed">
+    <joint name="base_joint" type="fixed">
         <origin xyz="0 0 0" rpy="0 0 0"/>
         <parent link="world"/>

Commit message: Camera Tracking updated.
More reliable. now limited by joint limits

File: dev_ws/src/trackingplatform/description/robot.urdf.xacro (robot description, xacro)
@@ -48,5 +48,5 @@
         <child link="azimuth_link"/>
         <axis xyz="0 0 1"/>
-        <limit lower="0" upper="${2*pi}" velocity="100" effort="100"/>
+        <limit lower="${-2*pi}" upper="${2*pi}" velocity="100" effort="100"/>
     </joint>
     <link name="azimuth_link">

File: dev_ws/src/trackingplatform/description/ros2_control.xacro (robot description, xacro)
@@ -6,18 +6,18 @@
         </hardware>
         <joint name="azimuth_joint">
-            <command_interface name="position">
-                <param name="min">-1</param>
-                <param name="max">1</param>
+            <command_interface name="velocity">
+                <param name="min">-10</param>
+                <param name="max">10</param>
             </command_interface>
             <state_interface name="position" />
-            <!-- <state_interface name="velocity" /> -->
+            <state_interface name="velocity" />
         </joint>
         <joint name="camera_joint">
-            <command_interface name="position">
-                <param name="min">-1</param>
-                <param name="max">1</param>
+            <command_interface name="velocity">
+                <param name="min">-10</param>
+                <param name="max">10</param>
             </command_interface>
-            <!-- <state_interface name="velocity" /> -->
             <state_interface name="position" />
+            <state_interface name="velocity" />
         </joint>
     </ros2_control>
