Commit message: Blobfind and camera subscriber working
ros2 run cv listener
must have the sim running

File: dev_ws/src/trackingplatform/description/gazebo.xacro (robot description, xacro)
@@ -65,5 +65,5 @@
             <visualize>true</visualize>
             <camera name="cam">
-                <horizontal_fov>1.3962634</horizontal_fov>
+                <horizontal_fov>0.2</horizontal_fov>
                 <image>
                     <width>640</width>

File: dev_ws/src/trackingplatform/description/robot.urdf.xacro (robot description, xacro)
@@ -31,10 +31,10 @@
             </material>
         </visual>
-        <collision>
+        <!-- <collision>
             <origin xyz="0 0 0.05" rpy="0 0 0"/>
             <geometry>
                 <box size="1 1 0.1" />
             </geometry>
-        </collision>
+        </collision> -->
         <inertial>
             <origin xyz="0 0 0.05" rpy="0 0 0"/>
@@ -50,5 +50,5 @@
         <limit lower="0" upper="${2*pi}" velocity="100" effort="100"/>
     </joint>
-        <link name="azimuth_link">
+    <link name="azimuth_link">
         <visual>
             <origin xyz="0 0 .2" rpy="0 0 0"/>
@@ -60,10 +60,10 @@
             </material>
         </visual>
-        <collision>
+        <!-- <collision>
             <origin xyz="0 0 0.05" rpy="0 0 0"/>
             <geometry>
                 <box size="1 1 0.1" />
             </geometry>
-        </collision>
+        </collision> -->
         <inertial>
             <origin xyz="0 0 0.05" rpy="0 0 0"/>
@@ -112,3 +112,5 @@
     </link>
    <xacro:include filename="gazebo.xacro" />
+<!-- Adding the Rocket -->
+   <xacro:include filename="rocket.urdf.xacro"/>
 </robot>

File: dev_ws/src/trackingplatform/description/rocket.urdf.xacro (robot description, xacro)
@@ -1,21 +1,97 @@
 <?xml version="1.0"?>
-<robot name="rocket">
-    <link name="base_link">
+<robot xmlns:xacro="http://www.ros.org/wiki/xacro" name="rocket">
+    <!-- <xacro:include filename="ros2_control.xacro" /> -->
+    <!-- <link name="world"></link>  Already made in main robot -->
+    <!-- <joint name="world_joint" type="planar">
+        <origin xyz="3 0 3" rpy="0 0 0"/>
+        <parent link="world"/>
+        <child link="rocket_link"/>
+        <axis xyz="1 0 0"/>
+        <limit lower="0" upper="100" velocity="100" effort="100"/>
+    </joint> -->
+    <link name="x_link">
+        <visual>
+            <origin xyz="0 0 0.05" rpy="0 0 0"/>
+            <geometry>
+                <cylinder length=".1" radius=".5" />
+            </geometry>
+            <material name="green">
+                <color rgba="0.2 1 0.2 1"/>
+            </material>
+        </visual>
+        <inertial>
+            <origin xyz="0 0 0.05" rpy="0 0 0"/>
+            <mass value="0.001" />
+            <inertia ixx="0.0" ixy="0.0" ixz="0.0" iyy="0.0" iyz="0.0" izz="0.0" />
+        </inertial>
     </link>
+    <!-- <link name="y_link">
+        <visual>
+            <origin xyz="0 0 0.05" rpy="0 0 0"/>
+            <geometry>
+                <cylinder length=".1" radius=".5" />
+            </geometry>
+            <material name="green">
+                <color rgba="0.2 1 0.2 1"/>
+            </material>
+        </visual>
+        <inertial>
+            <origin xyz="0 0 0.05" rpy="0 0 0"/>
+            <mass value="0.001" />
+            <inertia ixx="0.0" ixy="0.0" ixz="0.0" iyy="0.0" iyz="0.0" izz="0.0" />
+        </inertial>
+    </link>
+    <link name="xy_link">
+        <visual>
+            <origin xyz="0 0 0.05" rpy="0 0 0"/>
+            <geometry>
+                <cylinder length=".1" radius=".5" />
+            </geometry>
+            <material name="green">
+                <color rgba="0.2 1 0.2 1"/>
+            </material>
+        </visual>
+        <inertial>
+            <origin xyz="0 0 0.05" rpy="0 0 0"/>
+            <mass value="0.001" />
+            <inertia ixx="0.0" ixy="0.0" ixz="0.0" iyy="0.0" iyz="0.0" izz="0.0" />
+        </inertial>
+    </link> -->
+    <joint name="x" type="fixed">
+        <origin xyz="15 0 0" rpy="0 0 0"/>
+        <parent link="world"/>
+        <child link="x_link"/>
+        <axis xyz="1 0 0"/>
+        <limit lower="-100" upper="100" velocity="100" effort="100"/>
+    </joint>
+    <!-- <joint name="xy" type="fixed">
+        <origin xyz="0 0 0" rpy="0 0 0"/>
+        <parent link="x_link"/>
+        <child link="xy_link"/>
+    </joint>
+    <joint name="y" type="prismatic"> Breaks because Gazebo doesnt like "free" joints Maybe a 'fixed' buffer?
+        <origin xyz="0 0 1" rpy="0 0 0"/>
+        <parent link="x_link"/>
+        <child link="y_link"/>
+        <axis xyz="0 0 1"/>
+        <limit lower="0" upper="100" velocity="100" effort="100"/>
+    </joint> -->
     <joint name="rocket_joint" type="fixed">
-        <origin xyz="0 0 0" rpy="0 0 0"/>
-        <parent link="base_link"/>
-        <child link="rocket"/>
+        <origin xyz="0 0 1" rpy="0 ${pi/2} 0"/>
+        <parent link="x_link"/>
+        <child link="rocket_link"/>
+        <axis xyz="0 0 1"/>
+        <limit lower="0" upper="100" velocity="100" effort="100"/>
     </joint>
-    <link name="rocket">
+    <link name="rocket_link">
         <inertial>
-                    <origin xyz="0 0 0" rpy="0 0 0"/>
-                    <mass value="0.120" />
-                    <inertia ixx="7.58333333333e-06" ixy="0.0" ixz="0.0" iyy="7.58333333333e-06" iyz="0.0" izz="1.25e-05"/> <!-- This is actually wrong for this rocket -->
-                </inertial>
+            <origin xyz="0 0 0" rpy="0 0 0"/>
+            <mass value="0.120" />
+            <inertia ixx="7.58333333333e-06" ixy="0.0" ixz="0.0" iyy="7.58333333333e-06" iyz="0.0" izz="1.25e-05"/> <!-- This is actually wrong for this rocket -->
+        </inertial>
                 <collision>
-                    <origin rpy="0 0 0" xyz="0 0 0"/>
+                    <origin rpy="0 0 0" xyz="0 0 0.3"/>
                     <geometry>
-                        <box size="0.1 0.1 0.1"/>
+                        <box size="0.1 0.1 .6"/>
                     </geometry>
                 </collision>
@@ -31,12 +107,15 @@
                 </visual>
     </link>
-    <gazebo reference="rocket">
+    <gazebo reference="rocket_link">
         <material>Gazebo/Orange</material>
     </gazebo>
+  <gazebo reference="rocket_link">
+    <gravity>0</gravity>
+  </gazebo>
     <gazebo>
         <plugin name="gazebo_ros_joint_state_publisher"
             filename="libgazebo_ros_joint_state_publisher.so">
             <update_rate>20</update_rate>
-            <joint_name>rocket_joint</joint_name>
+            <joint_name>x</joint_name>
         </plugin>
     </gazebo>

Commit message: Camera Controller Implemeneted

File: dev_ws/src/trackingplatform/description/gazebo.xacro (robot description, xacro)
@@ -62,5 +62,5 @@
     <gazebo reference="camera_link">
         <sensor type="depth" name="my_camera">
-            <update_rate>20</update_rate>
+            <update_rate>60</update_rate>
             <visualize>true</visualize>
             <camera name="cam">

File: dev_ws/src/trackingplatform/description/rocket.urdf.xacro (robot description, xacro)
@@ -59,5 +59,5 @@
     </link> -->
     <joint name="x" type="fixed">
-        <origin xyz="15 0 0" rpy="0 0 0"/>
+        <origin xyz="15 5 0" rpy="0 0 0"/>
         <parent link="world"/>
         <child link="x_link"/>
@@ -77,9 +77,9 @@
         <limit lower="0" upper="100" velocity="100" effort="100"/>
     </joint> -->
-    <joint name="rocket_joint" type="fixed">
-        <origin xyz="0 0 1" rpy="0 ${pi/2} 0"/>
+    <joint name="rocket_joint" type="continuous">
+        <origin xyz="0 0 1" rpy="0 ${2*pi} 0"/>
         <parent link="x_link"/>
         <child link="rocket_link"/>
-        <axis xyz="0 0 1"/>
+        <axis xyz="1 0 0"/>
         <limit lower="0" upper="100" velocity="100" effort="100"/>
     </joint>
@@ -87,5 +87,5 @@
         <inertial>
             <origin xyz="0 0 0" rpy="0 0 0"/>
-            <mass value="0.120" />
+            <mass value="100.120" />
             <inertia ixx="7.58333333333e-06" ixy="0.0" ixz="0.0" iyy="7.58333333333e-06" iyz="0.0" izz="1.25e-05"/> <!-- This is actually wrong for this rocket -->
         </inertial>
@@ -97,5 +97,5 @@
                 </collision>
                 <visual>
-                    <origin rpy="1.5708 0 0" xyz="0 0 0"/>
+                    <origin rpy="1.5708 0 0" xyz="0 0 0.5"/>
                     <geometry>
                         <mesh filename="$(find trackingplatform)/models/Example.stl" scale="0.001 0.001 0.001"/>

Commit message: Updates

File: dev_ws/src/trackingplatform/description/gazebo.xacro (robot description, xacro)
@@ -27,7 +27,7 @@
         <plugin name="gazebo_ros_joint_state_publisher"
             filename="libgazebo_ros_joint_state_publisher.so">
-            <update_rate>20</update_rate>
+            <update_rate>60</update_rate>
             <joint_name>azimuth_joint</joint_name>
-            <joint_name>camera_joint</joint_name>
+            <joint_name>altitude_joint</joint_name>
         </plugin>
     </gazebo>
@@ -61,9 +61,9 @@
             try swapping "depth" to "camera"-->
     <gazebo reference="camera_link">
-        <sensor type="depth" name="my_camera">
+        <sensor type="camera" name="my_camera">
             <update_rate>60</update_rate>
             <visualize>true</visualize>
             <camera name="cam">
-                <horizontal_fov>0.2</horizontal_fov>
+                <horizontal_fov>.2</horizontal_fov>
                 <image>
                     <width>640</width>
@@ -75,9 +75,9 @@
                     <far>300</far>
                 </clip>
-                <noise>
+                <!-- <noise> This actually screws with the detection
                     <type>gaussian</type>
                     <mean>0.0</mean>
                     <stddev>0.007</stddev>
-                </noise>
+                </noise> -->
             </camera>
             <plugin name="camera_controller" filename="libgazebo_ros_camera.so">

File: dev_ws/src/trackingplatform/description/robot.urdf.xacro (robot description, xacro)
@@ -12,5 +12,5 @@
     <!-- The base origin is offset from the world origin. -->
     <joint name="base_joint" type="fixed">
-        <origin xyz="0 0 0" rpy="0 0 0"/>
+        <origin xyz="0 -10 0" rpy="0 0 0"/>
         <parent link="world"/>
         <child link="base_link"/>
@@ -43,5 +43,5 @@
         </inertial>
     </link>
-    <joint name="azimuth_joint" type="revolute">
+    <joint name="azimuth_joint" type="continuous">
         <origin xyz="0 0 0" rpy="0 0 0"/>
         <parent link="base_link"/>
@@ -75,10 +75,10 @@
     <!-- - Even though the camera isn't moving relative to the arm, it will probably be helpful to have its own link/frame rather than just adding more visuals to the arm -->
     <!-- - For this example, the camera_link origin will be at the centre of the camera's "sensor" -->
-    <joint name="camera_joint" type="revolute">
+    <joint name="altitude_joint" type="revolute">
         <origin xyz="0 0 1" rpy="0 0 0"/>
         <parent link="azimuth_link"/>
         <child link="camera_link"/>
         <axis xyz="0 -1 0"/>
-        <limit lower="0" upper="${pi/2}" velocity="100" effort="100"/>
+        <limit lower="0" upper="${pi}" velocity="100" effort="100"/>
     </joint>
     <!-- camera_link describes the camera at the end of the arm -->

File: dev_ws/src/trackingplatform/description/ros2_control.xacro (robot description, xacro)
@@ -13,5 +13,5 @@
             <state_interface name="velocity" />
         </joint>
-        <joint name="camera_joint">
+        <joint name="altitude_joint">
             <command_interface name="velocity">
                 <param name="min">-10</param>
